Commit message: change rear wheels

File: description/robot_core.xacro (robot description, xacro)
@@ -14,23 +14,26 @@
         <color rgba="0 0 0 1"/>
     </material>
+    <material name="yellow">
+        <color rgba="0.94 0.79 0.09 1"/>
+    </material>
     <!-- BASE LINK -->
     <link name="base_link">
     </link>
-    <!-- CHASSIS LINK -->
-    <joint name="chassis_joint" type="fixed">
+    <!-- BODY LINK -->
+    <joint name="body_joint" type="fixed">
         <parent link="base_link"/>
-        <child link="chassis"/>
-        <origin xyz="-0.023 0 0"/>
+        <child link="body"/>
+        <origin xyz="0.05 0 0"/>
     </joint>
-    <link name="chassis">
+    <link name="body">
         <visual>
-            <origin xyz="0.13 0 0.05"/>
+            <origin xyz="-0.135 0 0.05"/>
             <geometry>
                 <box size="0.27 0.1 0.1"/>
             </geometry>
-            <material name="white"/>
+            <material name="yellow"/>
         </visual>
         <collision>
-            <origin xyz="0.13 0 0.05"/>
+            <origin xyz="0 0 0"/>
             <geometry>
                 <box size="0.27 0.1 0.1"/>
@@ -41,15 +44,55 @@
         </xacro:inertial_box> -->
     </link>
-    <!-- LEFT WHEEL LINK -->
-    <joint name="left_wheel_joint" type="continuous">
+    <!-- LEFT REAR WHEEL LINK -->
+    <joint name="left_rear_wheel_joint" type="continuous">
         <parent link="base_link"/>
-        <child link="left_wheel"/>
-        <origin xyz="0 0.175 0" rpy="-${pi/2} 0 0"/>
+        <child link="left_rear_wheel"/>
+        <origin xyz="0 -0.05 0" rpy="-${pi/2} 0 0"/>
         <axis xyz="0 0 1"/>
     </joint>
-    <link name="left_wheel">
+    <link name="left_rear_wheel">
         <visual>
             <geometry>
-                <cylinder radius="0.1" length="0.01"/>
+                <cylinder radius="0.02" length="0.01"/>
+            </geometry>
+            <material name="black"/>
+        </visual>
+        <collision>
+            <geometry>
+                <cylinder radius="0.02" length="0.01"/>
+            </geometry>
+        </collision>
+    </link>
+    <!-- RIGHT REAR WHEEL LINK -->
+    <joint name="right_rear_wheel_joint" type="continuous">
+        <parent link="base_link"/>
+        <child link="right_rear_wheel"/>
+        <origin xyz="0 0.05 0" rpy="${pi/2} 0 0"/>
+        <axis xyz="0 0 -1"/>
+    </joint>
+    <link name="right_rear_wheel">
+        <visual>
+            <geometry>
+                <cylinder radius="0.02" length="0.01"/>
+            </geometry>
+            <material name="black"/>
+        </visual>
+        <collision>
+            <geometry>
+                <cylinder radius="0.02" length="0.01"/>
+            </geometry>
+        </collision>
+    </link>
+    <!-- LEFT FRONT WHEEL LINK
+    <joint name="left_front_wheel_joint" type="continuous">
+        <parent link="base_link"/>
+        <child link="left_rear_wheel"/>
+        <origin xyz="0 -0.05 0" rpy="-${pi/2} 0 0"/>
+        <axis xyz="0 0 1"/>
+    </joint>
+    <link name="left_rear_wheel">
+        <visual>
+            <geometry>
+                <cylinder radius="0.02" length="0.01"/>
             </geometry>
             <material name="blue"/>
@@ -57,22 +100,7 @@
         <collision>
             <geometry>
-                <cylinder radius="0.1" length="0.01"/>
+                <cylinder radius="0.02" length="0.01"/>
             </geometry>
         </collision>
-    </link>
-    <!-- RIGHT WHEEL LINK -->
-    <joint name="right_wheel_joint" type="continuous">
-        <parent link="base_link"/>
-        <child link="right_wheel"/>
-        <origin xyz="0 -0.175 0" rpy="${pi/2} 0 0"/>
-        <axis xyz="0 0 -1"/>
-    </joint>
-    <link name="right_wheel">
-        <visual>
-            <geometry>
-                <cylinder radius="0.1" length="0.01"/>
-            </geometry>
-            <material name="blue"/>
-        </visual>
-    </link>
+    </link> -->
 </robot>

Commit message: add front wheels and front stands

File: description/robot_core.xacro (robot description, xacro)
@@ -1,4 +1,8 @@
 <?xml version="1.0"?>
 <robot xmlns:xacro="http://www.ros.org/wiki/xacro" >
+<launch>
+    <node name="joint_state_publisher" pkg="joint_state_publisher" type="joint_state_publisher"/>
+    <node name="robot_state_publisher" pkg="robot_state_publisher" type="robot_state_publisher" output="screen"/>
+</launch>
     <!-- <xacro:include filename="inertial_macros.xacro"/> -->
     <material name="white">
@@ -23,10 +27,10 @@
     <joint name="body_joint" type="fixed">
         <parent link="base_link"/>
-        <child link="body"/>
-        <origin xyz="0.05 0 0"/>
-    </joint>
-    <link name="body">
-        <visual>
-            <origin xyz="-0.135 0 0.05"/>
+        <child link="body_link"/>
+        <origin xyz="0 0 0.02"/>
+    </joint>
+    <link name="body_link">
+        <visual>
+            <origin xyz="0.135 0 0.05"/>
             <geometry>
                 <box size="0.27 0.1 0.1"/>
@@ -35,5 +39,5 @@
         </visual>
         <collision>
-            <origin xyz="0 0 0"/>
+            <origin xyz="0.135 0 0.05"/>
             <geometry>
                 <box size="0.27 0.1 0.1"/>
@@ -44,9 +48,57 @@
         </xacro:inertial_box> -->
     </link>
+    <!-- CAMERA BASE LINK -->
+    <joint name="camera_base_joint" type="fixed">
+        <parent link="body_link"/>
+        <child link="camera_base_link"/>
+        <origin xyz="0.1 0 0.1"/>
+    </joint>
+    <link name="camera_base_link">
+        <visual>
+            <origin xyz="0.0275 0 0.0075"/>
+            <geometry>
+                <box size="0.055 0.035 0.015"/>
+            </geometry>
+            <material name="black"/>
+        </visual>
+        <collision>
+            <origin xyz="0.0275 0 0.0075"/>
+            <geometry>
+                <box size="0.055 0.035 0.015"/>
+            </geometry>
+        </collision>
+        <!-- <xacro:inertial_box mass="0.5" x="0.27" y="0.1" z="0.1"> -->
+            <!-- <origin xyz="0.13 0 0.05" rpy="0 0 0"/>
+        </xacro:inertial_box> -->
+    </link>
+    <!-- CAMERA BODY LINK -->
+    <joint name="camera_body_joint" type="fixed">
+        <parent link="camera_base_link"/>
+        <child link="camera_body_link"/>
+        <origin xyz="0.035 0 0.015"/>
+    </joint>
+    <link name="camera_body_link">
+        <visual>
+            <origin xyz="0.01 0 0.0175"/>
+            <geometry>
+                <box size="0.02 0.075 0.035"/>
+            </geometry>
+            <material name="black"/>
+        </visual>
+        <collision>
+            <origin xyz="0.01 0 0.0175"/>
+            <geometry>
+                <box size="0.02 0.075 0.035"/>
+            </geometry>
+        </collision>
+        <!-- <xacro:inertial_box mass="0.5" x="0.27" y="0.1" z="0.1"> -->
+            <!-- <origin xyz="0.13 0 0.05" rpy="0 0 0"/>
+        </xacro:inertial_box> -->
+    </link>
     <!-- LEFT REAR WHEEL LINK -->
     <joint name="left_rear_wheel_joint" type="continuous">
-        <parent link="base_link"/>
+        <parent link="body_link"/>
         <child link="left_rear_wheel"/>
-        <origin xyz="0 -0.05 0" rpy="-${pi/2} 0 0"/>
+        <origin xyz="0.05 -0.05 0" rpy="-${pi/2} 0 0"/>
         <axis xyz="0 0 1"/>
     </joint>
@@ -66,7 +118,7 @@
     <!-- RIGHT REAR WHEEL LINK -->
     <joint name="right_rear_wheel_joint" type="continuous">
-        <parent link="base_link"/>
+        <parent link="body_link"/>
         <child link="right_rear_wheel"/>
-        <origin xyz="0 0.05 0" rpy="${pi/2} 0 0"/>
+        <origin xyz="0.05 0.05 0" rpy="${pi/2} 0 0"/>
         <axis xyz="0 0 -1"/>
     </joint>
@@ -84,23 +136,87 @@
         </collision>
     </link>
-    <!-- LEFT FRONT WHEEL LINK
+    <!-- LEFT FRONT STAND LINK-->
+    <joint name="left_front_stand_joint" type="revolute">
+        <parent link="body_link"/>
+        <child link="left_front_stand_link"/>
+        <origin xyz="0.22 0.04 0" rpy="-${pi/2} 0 0"/>
+        <axis xyz="0 1 0"/>
+        <limit effort="1000.0" lower="-${pi/4}" upper="${pi/4}" velocity="0.5"/>
+    </joint>
+    <link name="left_front_stand_link">
+        <visual>
+            <origin xyz="0 0 0.005"/>
+            <geometry>
+                <cylinder radius="0.002" length="0.01"/>
+            </geometry>
+            <material name="blue"/>
+        </visual>
+        <collision>
+            <geometry>
+                <cylinder radius="0.002" length="0.01"/>
+            </geometry>
+        </collision>
+    </link>
+    <!-- RIGHT FRONT STAND LINK -->
+    <joint name="right_front_stand_joint" type="revolute">
+        <parent link="body_link"/>
+        <child link="right_front_stand_link"/>
+        <origin xyz="0.22 -0.04 0" rpy="${pi/2} 0 0"/>
+        <axis xyz="0 1 0"/>
+        <limit effort="1000.0" lower="${pi/4}" upper="-${pi/4}" velocity="0.5"/>
+    </joint>
+    <link name="right_front_stand_link">
+        <visual>
+            <origin xyz="0 0 0.005"/>
+            <geometry>
+                <cylinder radius="0.002" length="0.01"/>
+            </geometry>
+            <material name="blue"/>
+        </visual>
+        <collision>
+            <geometry>
+                <cylinder radius="0.002" length="0.01"/>
+            </geometry>
+        </collision>
+    </link>
+    <!-- LEFT FRONT WHEEL LINK -->
     <joint name="left_front_wheel_joint" type="continuous">
-        <parent link="base_link"/>
-        <child link="left_rear_wheel"/>
-        <origin xyz="0 -0.05 0" rpy="-${pi/2} 0 0"/>
+        <parent link="left_front_stand_link"/>
+        <child link="left_front_wheel"/>
+        <origin xyz="0 0 0.01" rpy="0 0 0"/>
         <axis xyz="0 0 1"/>
     </joint>
-    <link name="left_rear_wheel">
-        <visual>
-            <geometry>
-                <cylinder radius="0.02" length="0.01"/>
-            </geometry>
-            <material name="blue"/>
-        </visual>
-        <collision>
-            <geometry>
-                <cylinder radius="0.02" length="0.01"/>
-            </geometry>
-        </collision>
-    </link> -->
+    <link name="left_front_wheel">
+        <visual>
+            <geometry>
+                <cylinder radius="0.02" length="0.01"/>
+            </geometry>
+            <material name="black"/>
+        </visual>
+        <collision>
+            <geometry>
+                <cylinder radius="0.02" length="0.01"/>
+            </geometry>
+        </collision>
+    </link>
+    <!-- RIGHT FRONT WHEEL LINK -->
+    <joint name="right_front_wheel_joint" type="continuous">
+        <parent link="right_front_stand_link"/>
+        <child link="right_front_wheel"/>
+        <origin xyz="0 0 0.01" rpy="0 0 0"/>
+        <axis xyz="0 0 1"/>
+    </joint>
+    <link name="right_front_wheel">
+        <visual>
+            <geometry>
+                <cylinder radius="0.02" length="0.01"/>
+            </geometry>
+            <material name="black"/>
+        </visual>
+        <collision>
+            <geometry>
+                <cylinder radius="0.02" length="0.01"/>
+            </geometry>
+        </collision>
+    </link>
 </robot>

Commit message: add inertia

File: description/robot_core.xacro (robot description, xacro)
@@ -5,5 +5,5 @@
     <node name="robot_state_publisher" pkg="robot_state_publisher" type="robot_state_publisher" output="screen"/>
 </launch>
-    <!-- <xacro:include filename="inertial_macros.xacro"/> -->
+    <xacro:include filename="inertial_macros.xacro"/>
     <material name="white">
         <color rgba="1 1 1 1"/>
@@ -44,7 +44,7 @@
             </geometry>
         </collision>
-        <!-- <xacro:inertial_box mass="0.5" x="0.27" y="0.1" z="0.1"> -->
-            <!-- <origin xyz="0.13 0 0.05" rpy="0 0 0"/>
-        </xacro:inertial_box> -->
+        <xacro:inertial_box mass="0.5" x="0.27" y="0.1" z="0.1">
+            <origin xyz="0.13 0 0.05" rpy="0 0 0"/>
+        </xacro:inertial_box>
     </link>
     <!-- CAMERA BASE LINK -->
@@ -68,7 +68,7 @@
             </geometry>
         </collision>
-        <!-- <xacro:inertial_box mass="0.5" x="0.27" y="0.1" z="0.1"> -->
-            <!-- <origin xyz="0.13 0 0.05" rpy="0 0 0"/>
-        </xacro:inertial_box> -->
+        <xacro:inertial_box mass="0.05" x="0.055" y="0.035" z="0.015">
+            <origin xyz="0.0275 0 0.0075" rpy="0 0 0"/>
+        </xacro:inertial_box>
     </link>
     <!-- CAMERA BODY LINK -->
@@ -92,7 +92,7 @@
             </geometry>
         </collision>
-        <!-- <xacro:inertial_box mass="0.5" x="0.27" y="0.1" z="0.1"> -->
-            <!-- <origin xyz="0.13 0 0.05" rpy="0 0 0"/>
-        </xacro:inertial_box> -->
+        <xacro:inertial_box mass="0.05" x="0.02" y="0.075" z="0.035">
+            <origin xyz="0.01 0 0.0175" rpy="0 0 0"/>
+        </xacro:inertial_box>
     </link>
     <!-- LEFT REAR WHEEL LINK -->
@@ -115,4 +115,7 @@
             </geometry>
         </collision>
+        <xacro:inertial_cylinder mass="0.1" length="0.01" radius="0.02">
+            <origin xyz="0 0 0" rpy="0 0 0"/>
+        </xacro:inertial_cylinder>
     </link>
     <!-- RIGHT REAR WHEEL LINK -->
@@ -135,4 +138,7 @@
             </geometry>
         </collision>
+        <xacro:inertial_cylinder mass="0.1" length="0.01" radius="0.02">
+            <origin xyz="0 0 0" rpy="0 0 0"/>
+        </xacro:inertial_cylinder>
     </link>
     <!-- LEFT FRONT STAND LINK-->
@@ -157,4 +163,7 @@
             </geometry>
         </collision>
+        <xacro:inertial_cylinder mass="0.01" length="0.01" radius="0.002">
+            <origin xyz="0 0 0.005" rpy="0 0 0"/>
+        </xacro:inertial_cylinder>
     </link>
     <!-- RIGHT FRONT STAND LINK -->
@@ -179,4 +188,7 @@
             </geometry>
         </collision>
+        <xacro:inertial_cylinder mass="0.01" length="0.01" radius="0.002">
+            <origin xyz="0 0 0.005" rpy="0 0 0"/>
+        </xacro:inertial_cylinder>
     </link>
     <!-- LEFT FRONT WHEEL LINK -->
@@ -199,4 +211,7 @@
             </geometry>
         </collision>
+        <xacro:inertial_cylinder mass="0.1" length="0.01" radius="0.02">
+            <origin xyz="0 0 0" rpy="0 0 0"/>
+        </xacro:inertial_cylinder>
     </link>
     <!-- RIGHT FRONT WHEEL LINK -->
@@ -219,4 +234,7 @@
             </geometry>
         </collision>
+        <xacro:inertial_cylinder mass="0.1" length="0.01" radius="0.02">
+            <origin xyz="0 0 0" rpy="0 0 0"/>
+        </xacro:inertial_cylinder>
     </link>
 </robot>
